File: schematic/schematic.sch (KiCad schematic (older format))
At the start: 34 parts, among them J1 Signal_Input, J2 Conn_Power_Supply, J3 BNC, Q1 2N7000, U1 AD8021ARZ, U2 AD8021ARZ, U3 AD8021ARZ

Commit message: [Schematic] Use screw terminal for signal output
Parts:
- removed J3: BNC, symbol Connector:Conn_Coaxial
- added J3: Signal_Output, symbol Connector:Screw_Terminal_01x02
Connections:
- net GND: now also J3.2 (Pin_2)
- net at C15.1: now also J3.1 (Pin_1)
Changed lines of the file:
@@
 	9100 4900 9200 4900
-$Comp
-L Connector:Conn_Coaxial J3
-U 1 1 626B3B0A
-P 10800 5150
-F 0 "J3" H 10900 5125 50  0000 L CNN
-F 1 "BNC" H 10900 5034 50  0000 L CNN
-F 2 "" H 10800 5150 50  0001 C CNN
-F 3 " ~" H 10800 5150 50  0001 C CNN
-	1    10800 5150
-	1    0    0    -1
-$EndComp
-Wire Wire Line
-	10800 5350 10800 5400
-$Comp
-L power:GND #PWR031
-U 1 1 626B7ED1
-P 10800 5400
-F 0 "#PWR031" H 10800 5150 50  0001 C CNN
-F 1 "GND" H 10805 5227 50  0000 C CNN
-F 2 "" H 10800 5400 50  0001 C CNN
-F 3 "" H 10800 5400 50  0001 C CNN
-	1    10800 5400
-	1    0    0    -1
-$EndComp
 $Comp
 L Device:C C12
@@
 	8500 4900 8800 4900
 Connection ~ 8500 4900
-Wire Wire Line
-	10400 5150 10600 5150
 $Comp
 L power:GND #PWR01
@@
 	0    -1   1    0
 $EndComp
+$Comp
+L Connector:Screw_Terminal_01x02 J3
+U 1 1 6289B9DA
+P 10900 5150
+F 0 "J3" H 10850 5400 50  0000 L CNN
+F 1 "Signal_Output" H 10650 5300 50  0000 L CNN
+F 2 "" H 10900 5150 50  0001 C CNN
+F 3 "~" H 10900 5150 50  0001 C CNN
+	1    10900 5150
+	1    0    0    -1
+$EndComp
+$Comp
+L power:GND #PWR0101
+U 1 1 628A2484
+P 10650 5300
+F 0 "#PWR0101" H 10650 5050 50  0001 C CNN
+F 1 "GND" H 10655 5127 50  0000 C CNN
+F 2 "" H 10650 5300 50  0001 C CNN
+F 3 "" H 10650 5300 50  0001 C CNN
+	1    10650 5300
+	1    0    0    -1
+$EndComp
+Wire Wire Line
+	10650 5300 10650 5250
+Wire Wire Line
+	10650 5250 10700 5250
+Wire Wire Line
+	10400 5150 10700 5150
 $EndSCHEMATC

Commit message: [Schematic] Associate symbols with footprints
Parts:
- C1, C10, C12, C14, C15, C2, C6, C8: footprint (none) -> Capacitor_SMD:C_0603_1608Metric_Pad1.08x0.95mm_HandSolder
- C11, C13, C3, C5, C7, C9: value 100nF/5% -> 100nF/10%; footprint (none) -> Capacitor_SMD:C_0603_1608Metric_Pad1.08x0.95mm_HandSolder
- C4: value 6p8F -> 7pF/0.5pF; footprint (none) -> Capacitor_SMD:C_0603_1608Metric_Pad1.08x0.95mm_HandSolder
- J1, J3: footprint (none) -> TerminalBlock:TerminalBlock_bornier-2_P5.08mm
- J2: footprint (none) -> TerminalBlock:TerminalBlock_bornier-6_P5.08mm
- R1, R10, R11, R12, R2, R3, R4, R5, R6, R7, R8, R9: footprint (none) -> Resistor_SMD:R_0603_1608Metric_Pad0.98x0.95mm_HandSolder
- U1, U2, U3: footprint (none) -> Package_SO:SOIC-8_3.9x4.9mm_P1.27mm
Other:
- moved on the sheet: C3
