File: schematic/schematic.kicad_pcb (KiCad board)
At the start: 2 copper layers, 29.5 x 72.5 mm, 38 parts, among them J1 Signal_Input, J2 Conn_Power_Supply, J3 Signal_Output, Q1 2N7000, U1 AD8021ARZ, U2 AD8021ARZ, U3 AD8021ARZ

Commit message: [PCB] Flip power connector
Parts:
- moved J2 25.4 mm to (136.1, 110.0), turned to 90 degrees
- moved J1 5.08 mm to (136.1, 77.5), turned to 90 degrees
- moved J3 5.08 mm to (136.1, 122.3), turned to 90 degrees
Connections:
- J2 pad 1: +5V -> +12V
- J2 pad 2: -5V -> GND
- J2 pad 5: GND -> -5V
- J2 pad 6: +12V -> +5V
Routing:
- net Net-(C15-Pad1): track 15.1 -> 13.0 mm
- net Net-(C1-Pad2): track 17.9 -> 18.9 mm
Other:
- board text added: "+12V"
- board text added: "+5V"
- board text added: "-5V"
- board text added: "GND"
- board text added: "POWER"
- board text added: "Uin"
- board text added: "Uout"
